File: meterkast-friesland.sch (KiCad schematic (older format))
At the start: 0 parts

Commit message: Schema meterkast
Parts:
- added SW1: 63A, symbol Fuse_Box:4P1T
- added SW10, SW11: SW_SPDT, symbol Switch:SW_SPDT
- added SW2: 40A / 0,03A, symbol Fuse_Box:RCD_2P
- added SW3, SW5, SW6, SW7: 16A, symbol Fuse_Box:CB_2P
- added SW4: 25A / 0,03A, symbol Fuse_Box:RCD_2P_with_reset
- added SW8, SW9: 20A, symbol Fuse_Box:Relais_2P
Connections:
- new net: SW1.1, SW2.1 (L), SW4.2
- new net: SW1.7, SW2.3 (N), SW4.4
- new net: SW2.2 (L), SW3.1 (L)
- new net: SW2.4 (N), SW3.3 (N)
- new net: SW4.1, SW5.1 (L), SW6.1 (L), SW7.1 (L)
- new net: SW4.3, SW5.3 (N), SW6.3 (N), SW7.3 (N)
- new net A-1: SW8.1
- new net A-2: SW8.3
- new net A-L: SW5.2 (L), SW8.2, SW8.4
- new net A-N: SW5.4 (N)
- new net B-L: SW6.2 (L)
- new net B-N: SW6.4 (N)
- new net C-1: SW9.1
- new net C-10: SW10.3 (C), SW11.2 (B), SW8.5 (A1)
- new net C-11: SW11.3 (C), SW9.5 (A1)
- new net C-L: SW10.2 (B), SW7.2 (L), SW9.2
- new net C-N: SW7.4 (N), SW8.6 (A2), SW9.6 (A2)
- new net D-L: SW3.2 (L)
- new net D-N: SW3.4 (N)
- new net LINE: SW1.2
- new net NEUT: SW1.8
Other:
- note added: "A-1:\n* Buitenlamp kamer"
- note added: "A-2:\n* Binnenlamp kamer"
- note added: "A-L:\n* Meterkast\n* Woonkamer"
- note added: "B-L:\n* Gang\n* Buitendeur\n* Badkamer\n* WC\n* Keuken"
- note added: "C-1:\n* Buitenlamp schuur\n* Buitenlamp garage"
- note added: "C-L:\n* Slaapkamer 1\n* Slaapkamer 2\n* Schuur\n* Zolder"
- note added: "D-L:\n* Wasmachine schuur"
